File: cpu.kicad_sch (KiCad schematic)
At the start: 23 parts, among them SW1 Boot Select, U1 RP2040, U4 AP2112K-3.3, U5 W25Q16JVSS, X1 ABM8-272-T3

Commit message: prod version, I think
Parts:
- removed U4: AP2112K-3.3, Package_TO_SOT_SMD:SOT-23-5, symbol Regulator_Linear:AP2112K-3.3
- added C13: 1uF, Capacitor_SMD:C_0603_1608Metric, symbol Device:C_Small
- added C14, C15: 10uF, Capacitor_SMD:C_0805_2012Metric, symbol Device:C_Small
- added J3: Conn_01x03_Pin, Connector_PinHeader_2.54mm:PinHeader_1x03_P2.54mm_Vertical, symbol Connector:Conn_01x03_Pin
- added J5: Conn_01x04_Pin, Connector_PinHeader_2.54mm:PinHeader_1x04_P2.54mm_Vertical, symbol Connector:Conn_01x04_Pin
- added J7: Power, Connector_PinHeader_2.54mm:PinHeader_1x03_P2.54mm_Vertical, symbol Connector:Conn_01x03_Pin
- added SW2: Reset, Aaron:SW4_PTS815 SJM 250 SMTR LFS_CNK, symbol Switch:SW_Push
- added U4: XC6220B331MR, Package_TO_SOT_SMD:SOT-23-5, symbol Regulator_Linear:XC6220B331MR
- C1, C10, C11, C12, C2, C3, C4, C5, C6, C7, C8: footprint Capacitor_SMD:C_0805_2012Metric -> Capacitor_SMD:C_0603_1608Metric
- C9: value 0.1uF -> 1uF; footprint Capacitor_SMD:C_0805_2012Metric -> Capacitor_SMD:C_0603_1608Metric
- JP1: footprint (none) -> Jumper:SolderJumper-2_P1.3mm_Open_RoundedPad1.0x1.5mm
- R2, R3, R6: footprint Resistor_SMD:R_0805_2012Metric -> Resistor_SMD:R_0603_1608Metric
- R7, R8: footprint (none) -> Resistor_SMD:R_0603_1608Metric
- SW1: footprint (none) -> Aaron:SW4_PTS815 SJM 250 SMTR LFS_CNK
- U1: Digikey P/N (none) -> 2648-SC0914(13)CT-ND
- U5: Digikey P/N (none) -> 256-W25Q16JVUXIQTRCT-ND
- X1: footprint ABM8-272-T3_ABR -> Aaron:ABM8-272-T3_ABR
Connections:
- net +1V1: now also C13.2
- net +3.3V: now also C14.1, J7.3 (Pin_3), U4.5 (VOUT)
- net GND: now also C13.1, C14.2, C15.2, J3.2 (Pin_2), J7.2 (Pin_2), SW2.2, U4.2 (GND)
- net RESET: now also SW2.1
- net SWCLK: now also J3.3 (Pin_3)
- net SWD: now also J3.1 (Pin_1)
- net USB_VBUS: now also C15.1, J7.1 (Pin_1), U4.1 (VIN), U4.3 (CE)
- net IO8: now reaches U1.11 (GPIO8)
- net IO8: now also J5.4 (Pin_4)
- net IO5: now reaches U1.7 (GPIO5)
- net IO5: now also J5.1 (Pin_1)
- net IO6: now reaches U1.8 (GPIO6)
- net IO6: now also J5.2 (Pin_2)
- net IO7: now reaches U1.9 (GPIO7)
- net IO7: now also J5.3 (Pin_3)
Other:
- note removed: "ADC_AVDD"
